Commit message: Update urdf-rs version to support multiple visual/collision

File: sample.urdf (robot description, URDF)
Before this commit: robot robo, 13 links, 12 joints
Links:
- link root: geometry collision cylinder length=0.4 radius=0.1; visual box size=0.2 0.2 0.4

Commit message: Update nalgebra and k

File: sample.urdf (robot description, URDF)
Before this commit: robot robo, 13 links, 12 joints
Links:
- link l_wrist1: geometry visual cylinder length=0.2 radius=0.1
- link r_wrist1: geometry visual cylinder length=0.2 radius=0.1
- link root: geometry collision sphere radius=0.2; visual box size=0.2 0.2 0.4
